File: pcb/Swarm-B_20230626.kicad_pcb (KiCad board)
At the start: 2 copper layers, 81.8 x 72.1 mm, 29 parts, among them J1 5v_3Pi, J2 GND_3Pi, J3 RX_Break, J4 Conn_02x15_Top_Bottom, J5 I2C_3Pi, J6 3PI_SWTCH, J7 I2C_Exp, J8 ProxA, J9 ProxB, U1 74LS32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

Commit message: update
Routing:
- net +5V: track 120.3 -> 167.7 mm
Changed lines of the file:
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@@
   (segment (start 150.78055 73.297979) (end 142.134021 73.297979) (width 0.25) (layer "F.Cu") (net 29))
   (segment (start 142.134021 70.780021) (end 135.754 64.4) (width 0.25) (layer "F.Cu") (net 29))
+  (segment (start 149.657099 117.154044) (end 151.069956 117.154044) (width 0.25) (layer "F.Cu") (net 29))
   (segment (start 137.384 117.348) (end 137.384 112.298) (width 0.25) (layer "F.Cu") (net 29))
   (segment (start 135.209 75.063) (end 140.369 75.063) (width 0.25) (layer "F.Cu") (net 29))
@@
   (segment (start 132.209 82.11) (end 134.084 80.235) (width 0.25) (layer "F.Cu") (net 29))
   (segment (start 98.759652 119.333652) (end 96.774 117.348) (width 0.25) (layer "F.Cu") (net 29))
+  (segment (start 153.208587 115.015413) (end 153.208587 75.363596) (width 0.25) (layer "F.Cu") (net 29))
   (segment (start 134.084 80.235) (end 134.084 76.188) (width 0.25) (layer "F.Cu") (net 29))
   (segment (start 142.134021 73.297979) (end 140.369 75.063) (width 0.25) (layer "F.Cu") (net 29))
@@
   (segment (start 149.657099 117.154044) (end 137.577956 117.154044) (width 0.25) (layer "F.Cu") (net 29))
   (segment (start 134.084 76.188) (end 135.209 75.063) (width 0.25) (layer "F.Cu") (net 29))
+  (segment (start 151.069956 117.154044) (end 153.208587 115.015413) (width 0.25) (layer "F.Cu") (net 29))
   (segment (start 135.398348 119.333652) (end 98.759652 119.333652) (width 0.25) (layer "F.Cu") (net 29))
+  (segment (start 151.14297 73.297979) (end 150.78055 73.297979) (width 0.25) (layer "F.Cu") (net 29))
+  (segment (start 153.208587 75.363596) (end 151.14297 73.297979) (width 0.25) (layer "F.Cu") (net 29))
   (segment (start 132.209 82.933) (end 132.209 82.11) (width 0.25) (layer "F.Cu") (net 29))
   (segment (start 96.774 117.348) (end 92.648831 113.222831) (width 0.25) (layer "F.Cu") (net 29))

Commit message: update
Parts:
- moved U3 41.5 mm to (148.2, 97.0), turned to 90 degrees
- moved U2 41.3 mm to (121.3, 65.2), turned to 180 degrees
- moved R2 1.22 mm to (98.2, 125.4), turned to 150 degrees
- moved R3 0.71 mm to (95.7, 64.7), turned to 30 degrees
Routing:
- net Net-(D1-K): track 199.6 -> 0.00 mm
- net Net-(U2-OUT): track 186.6 -> 0.00 mm
- net +5V: track 167.7 -> 0.00 mm
- net Net-(A1-A0): track 102.1 -> 0.00 mm
- net Net-(D1-A): track 163.2 -> 61.4 mm
- net Net-(A1-A5): track 86.2 -> 0.00 mm
- net Net-(A1-A4): track 79.5 -> 0.00 mm
- net Net-(A1-A2): track 77.6 -> 0.00 mm
- net Net-(A1-D1/TX): track 73.6 -> 0.00 mm
- net Net-(J4-Pin_4): track 64.5 -> 0.00 mm
- net Net-(J4-Pin_2): track 59.3 -> 0.00 mm
- net Net-(A1-D4): track 53.5 -> 0.00 mm
- net Net-(A1-D3): track 51.9 -> 0.00 mm
- net Net-(A1-D2): track 46.5 -> 0.00 mm
- net Net-(A1-A1): track 39.1 -> 0.00 mm
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- removed copper zone on B.Cu, net GND
- removed copper zone on F.Cu, net GND
Other:
- rule pad_to_mask_clearance: 0.05 -> 0
- rule solder_mask_min_width: 0.1 -> 0.1016

Commit message: update
Routing:
- net Net-(D1-K): track 0.00 -> 186.8 mm
- net +5V: track 0.00 -> 174.6 mm
- net Net-(U2-OUT): track 0.00 -> 147.3 mm
- net Net-(D1-A): track 61.4 -> 188.8 mm
- net Net-(A1-A4): track 0.00 -> 83.8 mm
- net Net-(A1-D1/TX): track 0.00 -> 83.1 mm
- net Net-(A1-A5): track 0.00 -> 80.3 mm
- net Net-(A1-A2): track 0.00 -> 77.0 mm
- net Net-(A1-A0): track 0.00 -> 62.5 mm
- net Net-(A1-D4): track 0.00 -> 53.4 mm
- net Net-(A1-D3): track 0.00 -> 52.9 mm
- net Net-(J4-Pin_2): track 0.00 -> 51.7 mm
- net Net-(A1-D2): track 0.00 -> 40.4 mm
- net Net-(A1-A1): track 0.00 -> 40.2 mm
- net Net-(A1-D7): track 0.00 -> 27.9 mm
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- added copper zone on F.Cu, net GND

Commit message: update
Parts:
- removed D6: 1N5819, Diode_THT:D_DO-34_SOD68_P7.62mm_Horizontal
Connections:
- A1 pad 25: unconnected-(A1-A6-Pad25) -> Net-(A1-A6)
- A1 pad 26: unconnected-(A1-A7-Pad26) -> Net-(A1-A7)
- J1 pad 1: Net-(D6-K) -> +5V
- J1 pad 2: Net-(D6-K) -> +5V
- J4 pad 2: Net-(J4-Pin_2) -> unconnected-(J4-Pin_2-Pad2)
- J4 pad 4: Net-(J4-Pin_4) -> unconnected-(J4-Pin_4-Pad4)
- J8 pad 2: Net-(J4-Pin_2) -> Net-(A1-A7)
- J9 pad 2: Net-(J4-Pin_4) -> Net-(A1-A6)
Routing:
- net GND: track 0.00 -> 101.1 mm
- net Net-(A1-A6): track 0.00 -> 71.0 mm, vias 0 -> 1
- net Net-(A1-A7): track 0.00 -> 70.9 mm
- net Net-(A1-A2): track 77.0 -> 141.5 mm
- net Net-(J4-Pin_2): track 51.7 -> 0.00 mm
- net Net-(D1-A): track 188.8 -> 162.6 mm
- net Net-(J4-Pin_4): track 17.4 -> 0.00 mm
- net Net-(D1-K): track 186.8 -> 174.5 mm
- net Net-(D6-K): track 11.6 -> 0.00 mm
- net +5V: track 174.6 -> 184.7 mm
- net Net-(A1-D1/TX): track 83.1 -> 93.0 mm
- net Net-(A1-D4): track 53.4 -> 62.1 mm, vias 0 -> 1
- net Net-(A1-A4): track 83.8 -> 75.9 mm
- net Net-(A1-D2): track 40.4 -> 44.7 mm
- net Net-(U2-OUT): track 147.3 -> 143.8 mm
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- added copper zone on B.Cu, net GND
