File: pcb/Swarm-B_20230626.kicad_pcb (KiCad board)
At the start: 2 copper layers, 81.8 x 72.1 mm, 28 parts, among them J1 5v_3Pi, J2 GND_3Pi, J3 RX_Break, J4 Conn_02x15_Top_Bottom, J5 I2C_3Pi, J6 3PI_SWTCH, J7 I2C_Exp, J8 ProxA, J9 ProxB, U1 74LS32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

Commit message: update
Parts:
- added D5: IR_LED, LED_THT:LED_D3.0mm_Horizontal_O1.27mm_Z2.0mm, F.Cu at (145.5, 122.4)
- added D6: IR_LED, LED_THT:LED_D3.0mm_Horizontal_O1.27mm_Z2.0mm, F.Cu at (90.5, 120.6)
- added D7: IR_LED, LED_THT:LED_D3.0mm_Horizontal_O1.27mm_Z2.0mm, F.Cu at (147.2, 68.2)
- added D8: IR_LED, LED_THT:LED_D3.0mm_Horizontal_O1.27mm_Z2.0mm, F.Cu at (92.3, 66.2)
- moved D2 7.30 mm to (119.9, 62.0)
- moved D3 6.92 mm to (86.7, 93.0)
- moved D1 6.90 mm to (117.7, 126.3)
- moved D4 6.69 mm to (151.5, 95.8)
- moved J8 3.38 mm to (149.2, 72.0)
- moved J9 3.15 mm to (152.5, 109.5)
Routing:
- net GND: track 101.1 -> 0.00 mm
- net Net-(D1-K): track 174.5 -> 241.9 mm, vias 0 -> 2
- net Net-(A1-A2): track 141.5 -> 77.7 mm, vias 0 -> 1
- net Net-(D1-A): track 162.6 -> 213.6 mm
- net Net-(A1-A4): track 75.9 -> 99.9 mm, vias 0 -> 3
- net Net-(U2-OUT): track 143.8 -> 162.9 mm, vias 0 -> 3
- net Net-(A1-A5): track 82.8 -> 101.8 mm, vias 0 -> 1
- net Net-(A1-A7): track 70.9 -> 89.7 mm, vias 0 -> 1
- net Net-(A1-D1/TX): track 93.0 -> 75.3 mm, vias 0 -> 3
- net Net-(A1-A6): track 71.0 -> 57.4 mm, vias 1 -> 0
- net +5V: track 184.7 -> 175.1 mm, vias 0 -> 2
- net Net-(A1-D3): track 53.2 -> 44.3 mm, vias 2 -> 0
- net Net-(A1-D4): track 62.1 -> 55.5 mm, vias 1 -> 0
- net Net-(A1-A0): track 65.5 -> 62.7 mm
- net Net-(A1-D0/RX): track 8.46 -> 10.9 mm, vias 0 -> 1
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Other:
- board text added: "Dec 2024"
