File: pcb/Swarm-B_20230626.kicad_sch (KiCad schematic)
At the start: 29 parts, among them J1 5v_3Pi, J1 Conn_02x15_Top_Bottom, J2 GND_3Pi, J3 RX_Break, J5 I2C_3Pi, J6 3PI_SWTCH, J7 I2C_Exp, J8 ProxA, J9 ProxB, U1 74LS32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

Commit message: update
Parts:
- removed D6: 1N5819, Diode_THT:D_DO-34_SOD68_P7.62mm_Horizontal, symbol pspice:DIODE
Connections:
- net +5V: now also J1.1, J1.2
- net at A1.25 (A6): now also J9.2 (Pin_2)
- net at A1.26 (A7): now also J8.2 (Pin_2)
- net at J1.4 (Pin_4): no longer J9.2 (Pin_2)
- net at J1.2 (Pin_2): no longer J8.2 (Pin_2)
Changed lines of the file:
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@@
+    (stroke (width 0) (type default))
+  )
+  (wire (pts (xy 223.52 34.29) (xy 207.01 34.29))
     (stroke (width 0) (type default))
   )
@@
     (stroke (width 0) (type default))
   )
+  (wire (pts (xy 207.01 34.29) (xy 207.01 135.89))
+    (stroke (width 0) (type default))
+  )
   (wire (pts (xy 116.84 78.74) (xy 116.84 96.52))
     (stroke (width 0) (type default))
@@
     (stroke (width 0) (type default))
   )
+  (wire (pts (xy 207.01 135.89) (xy 191.77 135.89))
+    (stroke (width 0) (type default))
+  )
   (wire (pts (xy 257.81 72.39) (xy 257.81 76.2))
     (stroke (width 0) (type default))
@@
     (stroke (width 0) (type default))
   )
+  (wire (pts (xy 223.52 21.59) (xy 204.47 21.59))
+    (stroke (width 0) (type default))
+  )
   (wire (pts (xy 199.39 68.58) (xy 194.31 68.58))
     (stroke (width 0) (type default))
@@
     (stroke (width 0) (type default))
   )
+  (wire (pts (xy 204.47 21.59) (xy 204.47 138.43))
+    (stroke (width 0) (type default))
+  )
   (wire (pts (xy 181.61 146.05) (xy 179.07 146.05))
     (stroke (width 0) (type default))
@@
     (stroke (width 0) (type default))
   )
-  (wire (pts (xy 173.99 21.59) (xy 173.99 40.64))
-    (stroke (width 0) (type default))
-  )
   (wire (pts (xy 82.55 135.89) (xy 82.55 149.86))
     (stroke (width 0) (type default))
@@
     (stroke (width 0) (type default))
   )
-  (wire (pts (xy 175.26 34.29) (xy 223.52 34.29))
-    (stroke (width 0) (type default))
-  )
   (wire (pts (xy 257.81 123.19) (xy 257.81 128.27))
     (stroke (width 0) (type default))
@@
     (stroke (width 0) (type default))
   )
-  (wire (pts (xy 173.99 40.64) (xy 181.61 40.64))
-    (stroke (width 0) (type default))
-  )
   (wire (pts (xy 38.1 114.3) (xy 44.45 114.3))
     (stroke (width 0) (type default))
@@
     (stroke (width 0) (type default))
   )
-  (wire (pts (xy 175.26 34.29) (xy 175.26 45.72))
-    (stroke (width 0) (type default))
-  )
   (wire (pts (xy 59.69 132.08) (xy 59.69 138.43))
     (stroke (width 0) (type default))
   )
-  (wire (pts (xy 223.52 21.59) (xy 173.99 21.59))
-    (stroke (width 0) (type default))
-  )
   (wire (pts (xy 209.55 48.26) (xy 209.55 133.35))
     (stroke (width 0) (type default))
@@
     (stroke (width 0) (type default))
   )
-  (wire (pts (xy 175.26 45.72) (xy 181.61 45.72))
-    (stroke (width 0) (type default))
-  )
   (wire (pts (xy 270.51 137.16) (xy 270.51 135.89))
     (stroke (width 0) (type default))
@@
     (stroke (width 0) (type default))
   )
-  (wire (pts (xy 52.07 182.88) (xy 46.99 182.88))
+  (wire (pts (xy 46.99 182.88) (xy 62.23 182.88))
     (stroke (width 0) (type default))
   )
@@
   )
   (wire (pts (xy 181.61 38.1) (xy 171.45 38.1))
+    (stroke (width 0) (type default))
+  )
+  (wire (pts (xy 204.47 138.43) (xy 191.77 138.43))
     (stroke (width 0) (type default))
   )
@@
     )
   )
-  (symbol (lib_id "pspice:DIODE") (at 57.15 182.88 0) (unit 1)
-    (in_bom yes) (on_board yes) (dnp no)
-    (property "Reference" "D6" (at 57.15 176.149 0)
-      (effects (font (size 1.27 1.27)))
-    )
-    (property "Value" "1N5819" (at 57.15 178.4604 0)
-      (effects (font (size 1.27 1.27)))
-    )
-    (property "Footprint" "Diode_THT:D_DO-34_SOD68_P7.62mm_Horizontal" (at 57.15 182.88 0)
-      (effects (font (size 1.27 1.27)) hide)
-    )
-    (property "Datasheet" "~" (at 57.15 182.88 0)
-      (effects (font (size 1.27 1.27)) hide)
-    )
-    (pin "1")
-    (pin "2")
-    (instances
-      (project "Swarm-B_20230626"
-        (path "/2ef4a934-7614-4c51-b75c-13216ab373de"
-          (reference "D6") (unit 1)
-        )
-      )
-    )
-  )
   (symbol (lib_name "RESISTOR0402_2") (lib_id "SparkFun-Resistors:RESISTOR0402") (at 245.11 109.22 270) (unit 1)
     (in_bom yes) (on_board yes) (dnp no)
@@
       (effects (font (size 1.27 1.27)))
     )
-    (property "Value" "Conn_02x15_Top_Bottom" (at 187.96 34.8996 0)
-      (effects (font (size 1.27 1.27)))
-    )
+    (property "Value" "Conn_02x15_Top_Bottom" (at 187.96 30.48 0)
+      (effects (font (size 1.27 1.27)))
+    )

Commit message: update
Parts:
- added D5, D6, D7, D8: IR_LED, LED_THT:LED_D3.0mm_Horizontal_O1.27mm_Z2.0mm, symbol Device:LED
Connections:
- net at D1.1 (K), D2.1 (K), D3.1 (K)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: now also D5.1 (K), D6.1 (K), D7.1 (K), D8.1 (K)
- net at D1.2 (A), D2.2 (A), D3.2 (A)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: now also D5.2 (A), D6.2 (A), D7.2 (A), D8.2 (A)
Other:
- moved on the sheet: J1, J2
